File: pcb/ESP_RS/ESP_RS.kicad_sch (KiCad schematic)
At the start: 53 parts, among them J1 Conn_01x02, J2 USB_C_Receptacle_USB2.0_16P, J3 Conn_01x07_Socket, J4 Conn_02x05_Counter_Clockwise, Q1 SS8050, Q2 SS8050, U1 AMS1117-3.3, U2 TPS54202DDC, U3 CP2102N-Axx-xQFN28, U4 ESP32-WROOM-32E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

Commit message: d
Parts:
- removed C1, C13, C3, C8, C9: 22u, Capacitor_SMD:C_0603_1608Metric, symbol Device:C
- removed C10: 75p, Capacitor_SMD:C_0603_1608Metric, symbol Device:C
- removed C11, C12, C5: 0u1, Capacitor_SMD:C_0603_1608Metric, symbol Device:C
- removed C2: 10u, Capacitor_SMD:C_0805_2012Metric, symbol Device:C
- removed C4, C6: 0u1, Capacitor_SMD:C_0805_2012Metric, symbol Device:C
- removed C7: 4u7, Capacitor_SMD:C_0603_1608Metric, symbol Device:C
- removed D1: D_Schottky, Diode_SMD:D_SOD-323, symbol Device:D_Schottky
- removed D2, D4, D5: H5VL10B, Diode_SMD:D_SOD-882, symbol Device:D_TVS
- removed D3: LED, LED_SMD:LED_0603_1608Metric, symbol Device:LED
- removed J1: Conn_01x02, Connector_JST:JST_XH_B2B-XH-AM_1x02_P2.50mm_Vertical, symbol Connector_Generic:Conn_01x02
- removed J2: USB_C_Receptacle_USB2.0_16P, Connector_USB:USB_C_Receptacle_GCT_USB4105-xx-A_16P_TopMnt_Horizontal, symbol Connector:USB_C_Receptacle_USB2.0_16P
- removed J3: Conn_01x07_Socket, Connector_JST:JST_XH_B7B-XH-A_1x07_P2.50mm_Vertical, symbol Connector:Conn_01x07_Socket
- removed L1: SRN6045-150M, Inductor_SMD:L_Bourns_SRN6045TA, symbol Device:L
- removed Q1, Q2: SS8050, Package_TO_SOT_SMD:SOT-23, symbol Transistor_BJT:SS8050
- removed R1, R2: 5k1, Resistor_SMD:R_0603_1608Metric, symbol Device:R
- removed R10: 49.9, Resistor_SMD:R_0603_1608Metric, symbol Device:R
- removed R11, R33: 100k, Resistor_SMD:R_0603_1608Metric, symbol Device:R
- removed R12: 13k3, Resistor_SMD:R_0603_1608Metric, symbol Device:R
- removed R13, R3, R4: 10k, Resistor_SMD:R_0603_1608Metric, symbol Device:R
- removed R14, R15: 0, Resistor_SMD:R_0603_1608Metric, symbol Device:R
- removed R16: 2k1, Resistor_SMD:R_0603_1608Metric, symbol Device:R
- removed R34: 22k, Resistor_SMD:R_0603_1608Metric, symbol Device:R
- removed R5: 22k1, Resistor_SMD:R_0603_1608Metric, symbol Device:R
- removed R6: 510k, Resistor_SMD:R_0603_1608Metric, symbol Device:R
- removed R7: 47k5, Resistor_SMD:R_0603_1608Metric, symbol Device:R
- removed R8, R9: 2k, Resistor_SMD:R_0603_1608Metric, symbol Device:R
- removed U1: AMS1117-3.3, Package_TO_SOT_SMD:SOT-223-3_TabPin2, symbol Regulator_Linear:AMS1117-3.3
- removed U2: TPS54202DDC, Package_TO_SOT_SMD:SOT-23-6, symbol Regulator_Switching:TPS54202DDC
- removed U3: CP2102N-Axx-xQFN28, Package_DFN_QFN:QFN-28-1EP_5x5mm_P0.5mm_EP3.35x3.35mm, symbol Interface_USB:CP2102N-Axx-xQFN28
- removed U4: ESP32-WROOM-32E, RF_Module:ESP32-WROOM-32D, symbol RF_Module:ESP32-WROOM-32E
- J4: value Conn_02x05_Counter_Clockwise -> 02x05 IDC
Connections:
- net EN_P renamed ENABLE
- net OUT_P renamed OUT_5
- net PWR renamed SLEEP
- no-connect marks 19 -> 0
Other:
- added sheet ESP (esp.kicad_sch)
- added sheet PSU (PSU.kicad_sch)
- added sheet USB_UART (USB_UART.kicad_sch)
- moved on the sheet: H1, H2, H3, H4, J4, JP1, U5
