File: pcb/ESP_RS/eth.kicad_sch (KiCad schematic)
At the start: 36 parts, among them J5 RJ45_Kycon_G7LX-A88S7-BP-GY, U6 W5500, Y1 25 MHz

Commit message: d
Parts:
- renumbered R17 to R14, R18 to R15, R19 to R17, R20 to R18, R21 to R19, R22 to R20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
