File: pcb/ESP_RS/ESP_RS.kicad_pcb (KiCad board)
At the start: 2 copper layers, 45 x 74.8 mm, 87 parts, among them J1 Conn_01x02, J2 USB_C_Receptacle_USB2.0_16P, J3 Conn_01x07_Socket, J4 Conn_02x05_Counter_Clockwise, J5 RJ45_Kycon_G7LX-A88S7-BP-GY, Q1 SS8050, Q2 SS8050, U1 AMS1117-3.3, U2 TPS54202DDC, U3 CP2102N-Axx-xQFN28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

Commit message: v
Parts:
- removed J3: Conn_01x07_Socket, Connector_JST:JST_XH_B7B-XH-A_1x07_P2.50mm_Vertical
- removed J4: Conn_02x05_Counter_Clockwise, Connector_IDC:IDC-Header_2x05_P2.54mm_Horizontal
- removed JP1: 5V_EN, TestPoint:TestPoint_2Pads_Pitch2.54mm_Drill0.8mm
- removed R16: 2k1, Resistor_SMD:R_0603_1608Metric
- removed U5: 74LVC1G17, Package_TO_SOT_SMD:SOT-23-5
- added C30: 100n, Capacitor_SMD:C_0402_1005Metric, F.Cu at (164.3, 75.4)
- added J6: RJ45_LED_Shielded, Library:MTJ-88ARX1-FSM-PG-LH, F.Cu at (152.8, 127.3)
- added JP3: Jumper_2_Small_Open, PCM_4ms_SolderJumper:JUMPER_SMD_1x2_tiny, F.Cu at (161.4, 71.5)
- added JP4: Jumper_2_Small_Open, PCM_4ms_SolderJumper:JUMPER_SMD_1x2_tiny, F.Cu at (161.4, 73.6)
- added JP5: Jumper_2_Small_Open, PCM_4ms_SolderJumper:JUMPER_SMD_1x2_tiny, F.Cu at (161.4, 75.8)
- added R35: 0, Resistor_SMD:R_0603_1608Metric, F.Cu at (158.0, 65.1)
- added R36: 0, Resistor_SMD:R_0603_1608Metric, F.Cu at (158.0, 67.6)
- added R37: 120, Resistor_SMD:R_0603_1608Metric, F.Cu at (158.0, 70.1)
- added R38: 1k, Resistor_SMD:R_0402_1005Metric, F.Cu at (164.3, 71.4)
- added R39: 1k, Resistor_SMD:R_0402_1005Metric, F.Cu at (164.3, 73.4)
- added U7: SN65HVD1781, Package_SO:SOIC-8_3.9x4.9mm_P1.27mm, F.Cu at (164.3, 67.2)
Connections:
- U4 pad 10: Net-(J3-Pin_2) -> unconnected-(U4-IO25-Pad10)
- U4 pad 11: Net-(J3-Pin_3) -> unconnected-(U4-IO26-Pad11)
- U4 pad 12: Net-(J3-Pin_4) -> unconnected-(U4-IO27-Pad12)
- U4 pad 28: /OUT -> /RE/DE
- U4 pad 30: /R2 -> unconnected-(U4-IO18-Pad30)
- U4 pad 31: /R1 -> unconnected-(U4-IO19-Pad31)
- U4 pad 33: /SDA -> /RX
- U4 pad 36: /SCL -> /TX
- U4 pad 8: Net-(J3-Pin_5) -> unconnected-(U4-IO32-Pad8)
- U4 pad 9: Net-(J3-Pin_6) -> unconnected-(U4-IO33-Pad9)
Routing:
- net /SCL: track 41.5 -> 0.00 mm, vias 2 -> 0
- net /TX: track 16.1 -> 57.6 mm, vias 2 -> 4
- net unconnected-(U4-IO18-Pad30): track 0.00 -> 40.1 mm, vias 0 -> 2
- net /R2: track 40.1 -> 0.00 mm, vias 2 -> 0
- net /SDA: track 33.3 -> 0.00 mm, vias 2 -> 0
- net /RX: track 13.6 -> 46.9 mm, vias 2 -> 4
- net unconnected-(U4-IO19-Pad31): track 0.00 -> 29.9 mm, vias 0 -> 2
- net /R1: track 29.9 -> 0.00 mm, vias 2 -> 0
- net unconnected-(U4-IO33-Pad9): track 0.00 -> 26.7 mm, vias 0 -> 1
- net Net-(J3-Pin_6): track 26.7 -> 0.00 mm, vias 1 -> 0
- net unconnected-(U4-IO32-Pad8): track 0.00 -> 26.4 mm, vias 0 -> 1
- net Net-(J3-Pin_5): track 26.4 -> 0.00 mm, vias 1 -> 0
- net /RE/DE: track 0.00 -> 19.9 mm, vias 0 -> 2
- net /OUT: track 19.9 -> 0.00 mm, vias 2 -> 0
- net unconnected-(U4-IO27-Pad12): track 0.00 -> 19.8 mm
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