File: pcb/RaSens/RaSens.kicad_pcb (KiCad board)
At the start: 2 copper layers, 167 x 48 mm, 57 parts, among them J1 TBP04R12-500-04BE, J2 TBP04R12-500-04BE, J3 Conn_02x05_Counter_Clockwise, J6 TBP04R12-500-02BE, K1 SHV05-1A85-78L2K, K2 SHV05-1A85-78L2K, K3 SHV05-1A85-78L2K, K4 SHV05-1A85-78L2K, K5 DIP12-1A72-11L, Q11 2N2222A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

Commit message: V5
Parts:
- removed C10: 100n, Capacitor_SMD:C_0805_2012Metric
- removed C14: 250p, Capacitor_SMD:C_1206_3216Metric
- removed D16, D20, D21, D22: UF4007, Diode_THT:D_DO-41_SOD81_P10.16mm_Horizontal
- removed D23, D24: BAS21, Diode_SMD:D_SMA-SMB_Universal_Handsoldering
- removed Q11, Q12, Q13, Q14: 2N2222A, Package_TO_SOT_THT:TO-92L_Inline
- removed R25: 200k, Resistor_SMD:R_0805_2012Metric
- removed R26: 2Meg, Resistor_SMD:R_0805_2012Metric
- removed R27: 3Meg, Resistor_SMD:R_0805_2012Metric
- removed R34: 1k, Resistor_SMD:R_0603_1608Metric
- removed U3: LM311, Package_DIP:DIP-8_W7.62mm_Socket
- added D1: 1N5819WS, Diode_SMD:D_SOD-323, B.Cu at (203.5, 101.3)
- added D3: 1N5819WS, Diode_SMD:D_SOD-323, B.Cu at (203.5, 94.9)
- added D4: 1N5819WS, Diode_SMD:D_SOD-323, B.Cu at (203.5, 88.5)
- added D5: 1N5819WS, Diode_SMD:D_SOD-323, B.Cu at (203.5, 82.1)
- added J5: Conn_01x02, Connector_JST:JST_XH_B2B-XH-A_1x02_P2.50mm_Vertical, F.Cu at (105.8, 75.7)
- added Q1: MMBT2222A, Package_TO_SOT_SMD:SOT-23, F.Cu at (211.5, 107.4)
- added Q2: MMBT2222A, Package_TO_SOT_SMD:SOT-23, F.Cu at (207.9, 107.4)
- added Q3: MMBT2222A, Package_TO_SOT_SMD:SOT-23, F.Cu at (200.7, 107.4)
- added Q4: MMBT2222A, Package_TO_SOT_SMD:SOT-23, F.Cu at (204.3, 107.4)
- added U2: COMPARATOR, Library:COMPARATOR, F.Cu at (181.0, 112.4)
- J6: value TBP04R12-500-02BE -> Conn_01x02; footprint Connector_Phoenix_MSTB:PhoenixContact_MSTBA_2,5_2-G-5,08_1x02_P5.08mm_Horizontal -> Connector_JST:JST_XH_B2B-XH-A_1x02_P2.50mm_Vertical
- moved R31 16.0 mm to (203.8, 111.1)
- moved J6 8.79 mm to (116.0, 75.7), turned to 0 degrees
- moved R29 7.78 mm to (207.4, 111.1)
- moved R30 7.39 mm to (200.2, 111.1)
- moved R45 6.15 mm to (211.0, 111.1)
- moved K1 6.10 mm to (203.5, 82.1)
- moved K4 4.70 mm to (203.5, 101.3)
- moved K2 2.50 mm to (203.5, 88.5)
- moved K3 1.10 mm to (203.5, 94.9)
Connections:
- J6 pad 1: GND -> Net-(D25-K)
- J6 pad 2: Net-(D25-K) -> GND
Routing:
- net +3.3V: track 127.7 -> 54.1 mm, vias 6 -> 4
- net +5V: track 235.1 -> 191.1 mm, vias 2 -> 3
- net Net-(D5-A): track 46.2 -> 28.1 mm
- net /GEIGER_OUTPUT: track 109.7 -> 127.2 mm
- net /SW3: track 56.4 -> 73.4 mm
- net Net-(D1-A): track 23.8 -> 7.37 mm, vias 1 -> 0
- net Net-(D4-A): track 34.8 -> 20.2 mm, vias 1 -> 0
- net Net-(D3-A): track 27.5 -> 15.3 mm, vias 1 -> 0
- net /tube_sel-dsch/TUBE+: track 53.1 -> 42.3 mm
- net Net-(D23-A): track 10.3 -> 0.00 mm
- net /SW2: track 116.6 -> 125.9 mm
- net /SW1: track 125.0 -> 131.3 mm
- net Net-(J1-Pin_1): track 20.2 -> 16.6 mm
- net Net-(J1-Pin_4): track 18.4 -> 14.9 mm
- net Net-(C13-Pad2): track 16.1 -> 19.6 mm
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- added copper zone on B.Cu, net Net-(D25-K)
Other:
- board text added: "RaSens V5"
- board text removed: "RaSens V4.1"
