File: pcb/RaSens/RaSens.kicad_sch (KiCad schematic)
At the start: 39 parts, among them J3 Conn_02x05_Counter_Clockwise, J6 TBP04R12-500-02BE, K5 DIP12-1A72-11L, Q15 2N2222A, T1 GA3460-BL, U1 Switcher, U3 LM311

Commit message: V5
Parts:
- removed C10: 100n, Capacitor_SMD:C_0805_2012Metric, symbol Device:C
- removed C14: 250p, Capacitor_SMD:C_1206_3216Metric, symbol Device:C
- removed D23, D24: BAS21, Diode_SMD:D_SMA-SMB_Universal_Handsoldering, symbol Device:D
- removed J6: TBP04R12-500-02BE, Connector_Phoenix_MSTB:PhoenixContact_MSTBA_2,5_2-G-5,08_1x02_P5.08mm_Horizontal, symbol Connector:Screw_Terminal_01x02
- removed R25: 200k, Resistor_SMD:R_0805_2012Metric, symbol Device:R
- removed R26: 2Meg, Resistor_SMD:R_0805_2012Metric, symbol Device:R
- removed R27: 3Meg, Resistor_SMD:R_0805_2012Metric, symbol Device:R
- removed R34: 1k, Resistor_SMD:R_0603_1608Metric, symbol Device:R
- removed U3: LM311, Package_DIP:DIP-8_W7.62mm_Socket, symbol Comparator:LM311
- added J5, J6: Conn_01x02, Connector_JST:JST_XH_B2B-XH-A_1x02_P2.50mm_Vertical, symbol Connector_Generic:Conn_01x02
- added U2: COMPARATOR, Library:COMPARATOR, symbol library:Comparator
Connections:
- net +5V: now also U2.1 (+5V)
- net GEIGER_OUTPUT: now also U2.3 (OUT)
- net GND: now also J5.2 (Pin_2), J6.2 (Pin_2), U2.4 (GND)
- net at C13.2: now also U2.5 (IN), U2.6 (IN), U2.7 (IN), U2.8 (IN)
- net at D25.1 (K), K5.1, K5.14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: now also J5.1 (Pin_1), J6.1 (Pin_1)
- no-connect marks 2 -> 1

Commit message: d
Other:
- title: Geiger Counter Module -> RaSens Pro
Changed lines of the file:
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@@
 	(paper "A4")
 	(title_block
-		(title "Geiger Counter Module")
-		(date "2025-09-16")
-		(rev "A")
+		(title "RaSens Pro")
+		(date "2026-05-17")
+		(rev "v5")
 	)
 	(junction
