File: pcb/RaSens/tube_sel-dsch.kicad_sch (KiCad schematic)
At the start: 18 parts, among them J1 TBP04R12-500-04BE, J2 TBP04R12-500-04BE, K1 SHV05-1A85-78L2K, K2 SHV05-1A85-78L2K, K3 SHV05-1A85-78L2K, K4 SHV05-1A85-78L2K, Q11 2N2222A, Q12 2N2222A, Q13 2N2222A, Q14 2N2222A

Commit message: V5
Parts:
- removed D16, D20, D21, D22: UF4007, Diode_THT:D_DO-41_SOD81_P10.16mm_Horizontal, symbol Diode:BA157
- removed Q11, Q12, Q13, Q14: 2N2222A, Package_TO_SOT_THT:TO-92L_Inline, symbol Transistor_BJT:BC107
- added D1, D3, D4, D5: 1N5819WS, Diode_SMD:D_SOD-323, symbol Diode:1N5819WS
- added Q1, Q2, Q3, Q4: MMBT2222A, Package_TO_SOT_SMD:SOT-23, symbol Transistor_BJT:MMBT2222A
Connections:
- net +5V: now also D1.1 (K), D3.1 (K), D4.1 (K), D5.1 (K)
- net GND: now also Q1.2 (E), Q2.2 (E), Q3.2 (E), Q4.2 (E)
- net at R29.1: now also Q2.1 (B)
- net at K2.5: now also D4.2 (A), Q2.3 (C)
- net at R30.1: now also Q3.1 (B)
- net at K3.5: now also D3.2 (A), Q3.3 (C)
- net at R31.1: now also Q4.1 (B)
- net at K4.5: now also D1.2 (A), Q4.3 (C)
- net at K1.5: now also D5.2 (A), Q1.3 (C)
- net at R45.1: now also Q1.1 (B)

Commit message: d
Other:
- title: (none) -> RaSens Pro
Changed lines of the file:
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@@
 	(paper "A4")
 	(title_block
-		(date "2025-09-16")
+		(title "RaSens Pro")
+		(date "2026-05-17")
+		(rev "v5")
 	)
 	(junction
