File: pcb/RaSensLite/RaSensLite.kicad_pcb (KiCad board)
At the start: 2 copper layers, 100 x 48 mm, 78 parts, among them J1 TBP04R12-500-04BE, J2 TBP04R12-500-04BE, J3 Conn_02x05_Counter_Clockwise, J4 TC2030, J6 TBP04R12-500-02BE, K5 DIP12-1A72-11L, Q1 IPP075N15N3, Q15 2N2222A, U2 DA2032-AL, U3 LM311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

Commit message: V5
Parts:
- removed C10: 100n, Capacitor_SMD:C_0805_2012Metric
- removed C14: 250p, Capacitor_SMD:C_1206_3216Metric
- removed C8: EFDKA1CK105D032LH, Capacitor_THT:C_Rect_L31.5mm_W11.0mm_P27.50mm_MKS4
- removed D23, D24: BAS21, Diode_SMD:D_SOD-123F
- removed R25: 200k, Resistor_SMD:R_0805_2012Metric
- removed R26: 2Meg, Resistor_SMD:R_0805_2012Metric
- removed R27: 3Meg, Resistor_SMD:R_0805_2012Metric
- removed R34: 1k, Resistor_SMD:R_0603_1608Metric
- removed U3: LM311, Package_DIP:DIP-8_W7.62mm_Socket
- added C2: ECW-FD2J105PQ, Capacitor_THT:C_Rect_L18.0mm_W7.0mm_P15.00mm_FKS3_FKP3, F.Cu at (150.5, 74.4)
- added J5: Conn_01x02, Connector_JST:JST_XH_B2B-XH-A_1x02_P2.50mm_Vertical, F.Cu at (80.0, 88.2)
- added U1: COMPARATOR, Library:COMPARATOR, F.Cu at (149.2, 105.4)
- D3: value STATUS1 -> STATUS2
- J6: value TBP04R12-500-02BE -> Conn_01x02; footprint Connector_Phoenix_MSTB:PhoenixContact_MSTBA_2,5_2-G-5,08_1x02_P5.08mm_Horizontal -> Connector_JST:JST_XH_B2B-XH-A_1x02_P2.50mm_Vertical
- moved J6 9.22 mm to (72.9, 88.2), turned to 90 degrees
- moved R35 2.50 mm to (81.3, 93.4)
- moved R36 2.50 mm to (83.8, 93.4)
Connections:
- J3 pad 10: /SDA -> /SCL
- J3 pad 9: /SCL -> /SDA
- J6 pad 1: GND -> Net-(D25-K)
- J6 pad 2: Net-(D25-K) -> GND
Routing:
- net +5V: track 260.5 -> 216.8 mm, vias 13 -> 11
- net +3.3V: track 36.9 -> 18.6 mm, vias 3 -> 1
- net Net-(C13-Pad2): track 22.9 -> 10.5 mm
- net GND: track 42.9 -> 37.1 mm, vias 44 -> 42
- net Net-(D23-A): track 5.24 -> 0.00 mm
- net /SDA: track 13.7 -> 11.2 mm
- net /SCL: track 12.4 -> 14.1 mm, vias 2 -> 0
- net /GEIGER_OUTPUT: track 90.1 -> 88.9 mm
Other:
- board text added: "GND"
- board text added: "RaSensLite V5"
- board text removed: "RaSensLite V1.0"
