File: pcb/RaSensLite/RaSensLite.kicad_pcb (KiCad board)
At the start: 2 copper layers, 100 x 48 mm, 71 parts, among them J1 TBP04R12-500-04BE, J2 TBP04R12-500-04BE, J3 Conn_02x05_Counter_Clockwise, J4 TC2030, J5 Conn_01x02, J6 Conn_01x02, K5 DIP12-1A72-11L, Q1 IPP075N15N3, Q15 2N2222A, U1 COMPARATOR, U2 DA2032-AL, U4 LM4040DBZ-2.5, U5 ATmega328P-A, U6 LM317_SOT-223, U7 LM321, U8 TC4420, U9 LM321

Commit message: v
Parts:
- removed C11: 1u, Capacitor_SMD:C_0603_1608Metric
- removed the C12 at (96.2, 111.8)
- removed D25: UF4007, Diode_THT:D_DO-41_SOD81_P10.16mm_Horizontal
- removed the J1 at (160.0, 91.1)
- removed K5: DIP12-1A72-11L, Relay_THT:Relay_StandexMeder_DIP_LowProfile
- removed Q15: 2N2222A, Package_TO_SOT_THT:TO-92L_Inline
- removed the R17 at (97.8, 109.1)
- removed the R18 at (96.3, 109.1)
- removed R46: 1k, Resistor_SMD:R_0805_2012Metric
- removed the U6 at (103.1, 110.9)
- added C10: EEE-FN1C102UP, Capacitor_SMD:CP_Elec_10x10.5, F.Cu at (100.7, 77.8)
- added C2: 2n2, Capacitor_SMD:C_0603_1608Metric, F.Cu at (108.3, 78.5)
- added C21: 100n, Capacitor_SMD:C_0402_1005Metric, F.Cu at (159.9, 102.3)
- added C22: 100p, Capacitor_SMD:C_0603_1608Metric, F.Cu at (155.1, 100.3)
- added C23: 0u1, Capacitor_SMD:C_0402_1005Metric, F.Cu at (151.1, 93.9)
- added C24: 1u, Capacitor_SMD:C_0402_1005Metric, F.Cu at (105.6, 87.8)
- added C25: 22u, Capacitor_SMD:C_1206_3216Metric, F.Cu at (103.8, 84.9)
- added C26: 10p, Capacitor_SMD:C_0603_1608Metric, F.Cu at (103.0, 90.3)
- added C27: 100n, Capacitor_SMD:C_0402_1005Metric, F.Cu at (107.1, 84.7)
- added C28: 22u, Capacitor_SMD:C_1206_3216Metric, F.Cu at (100.2, 86.0)
- added C7: 100n, Capacitor_SMD:C_0402_1005Metric, F.Cu at (88.5, 89.0)
- added D7: D_Schottky, Diode_SMD:D_SOD-323, F.Cu at (159.5, 111.1)
- added D8: 1N5819WS, Diode_SMD:D_SOD-323, F.Cu at (145.1, 94.0)
- added D9: 1N5819WS, Diode_SMD:D_SOD-323, F.Cu at (148.5, 94.0)
- added J2: RJ45_LED_Shielded, Library:MTJ-88ARX1-FSM-PG-LH, F.Cu at (77.3, 86.5)
- added JP2: Jumper_2_Small_Open, PCM_4ms_SolderJumper:JUMPER_SMD_1x2_tiny, F.Cu at (84.9, 91.1)
- added JP3: Jumper_2_Small_Open, PCM_4ms_SolderJumper:JUMPER_SMD_1x2_tiny, F.Cu at (84.9, 79.5)
- added JP4: Jumper_2_Small_Open, PCM_4ms_SolderJumper:JUMPER_SMD_1x2_tiny, F.Cu at (85.9, 87.5)
- added JP5: Jumper_2_Small_Open, PCM_4ms_SolderJumper:JUMPER_SMD_1x2_tiny, F.Cu at (113.1, 77.5)
- added JP6: Jumper_2_Open, TestPoint:TestPoint_2Pads_Pitch2.54mm_Drill0.8mm, F.Cu at (157.9, 97.5)
- added JP7: Jumper_2_Small_Open, PCM_4ms_SolderJumper:JUMPER_SMD_1x2_tiny, F.Cu at (91.7, 92.2)
- added JP8: Jumper_2_Small_Open, PCM_4ms_SolderJumper:JUMPER_SMD_1x2_tiny, F.Cu at (87.8, 92.2)
- added L1: LSANB2016KKT4R7M, Inductor_SMD:L_0805_2012Metric, F.Cu at (103.3, 87.0)
- added R10: 120, Resistor_SMD:R_0603_1608Metric, F.Cu at (85.9, 85.1)
- added R2: 1k, Resistor_SMD:R_0402_1005Metric, F.Cu at (84.9, 93.0)
- added R29: 1k, Resistor_SMD:R_0402_1005Metric, F.Cu at (156.4, 100.9)
- added R3: 1k, Resistor_SMD:R_0402_1005Metric, F.Cu at (84.9, 81.4)
- added R30: 470, Resistor_SMD:R_0402_1005Metric, F.Cu at (156.2, 110.3)
- added R31: 330k, Resistor_SMD:R_0402_1005Metric, F.Cu at (158.5, 100.9)
- added R32: 1Meg, Resistor_SMD:R_0402_1005Metric, F.Cu at (157.5, 100.9)
- added R33: 1M, Resistor_SMD:R_0402_1005Metric, F.Cu at (153.7, 93.9)
- added R34: 100k, Resistor_SMD:R_0402_1005Metric, F.Cu at (153.0, 98.7)
- added R35: 10k, Resistor_SMD:R_0402_1005Metric, F.Cu at (151.0, 98.7)
- added R36: 59k, Resistor_SMD:R_0603_1608Metric, F.Cu at (148.6, 92.2)
- added R37: 100k, Resistor_SMD:R_0402_1005Metric, F.Cu at (146.0, 92.2)
- added R38: 10, Resistor_SMD:R_0402_1005Metric, F.Cu at (107.1, 88.7)
- added R39: 47k, Resistor_SMD:R_0402_1005Metric, F.Cu at (107.1, 89.7)
- added R40: 7k68, Resistor_SMD:R_0603_1608Metric, F.Cu at (105.3, 90.3)
- added R41: 40k2, Resistor_SMD:R_0603_1608Metric, F.Cu at (103.0, 88.7)
- added R42: 100k, Resistor_SMD:R_0402_1005Metric, F.Cu at (107.1, 85.7)
- added R7: 0, Resistor_SMD:R_0603_1608Metric, F.Cu at (97.1, 86.8)
- added R8: 0, Resistor_SMD:R_0603_1608Metric, F.Cu at (97.1, 85.2)
- added RV1: 3314J-1-504E, Potentiometer_SMD:Potentiometer_Bourns_3314J_Vertical, F.Cu at (146.7, 97.6)
- added SW1: SW_DIP_x04, Button_Switch_SMD:SW_DIP_SPSTx04_Slide_6.7x11.72mm_W6.73mm_P2.54mm_LowProfile_JPin, F.Cu at (102.0, 113.1)
- added U10: ATtiny412-SS, Package_SO:SOIC-8_3.9x4.9mm_P1.27mm, F.Cu at (156.9, 105.6)
- added U11: LT1711xMS8, Package_SO:MSOP-8_3x3mm_P0.65mm, F.Cu at (153.5, 96.2)
- added U12: MP1476, Package_TO_SOT_SMD:SOT-563, F.Cu at (107.4, 87.2)
- added U3: SN65HVD1781, Package_SO:SOIC-8_3.9x4.9mm_P1.27mm, F.Cu at (91.8, 85.9)
- C12: renamed from C6; footprint Capacitor_SMD:C_0603_1608Metric -> Capacitor_SMD:C_0402_1005Metric
- C13: renamed from C9; footprint Capacitor_SMD:C_0603_1608Metric -> Capacitor_SMD:C_0402_1005Metric
- C14: renamed from C1; footprint Capacitor_SMD:C_0603_1608Metric -> Capacitor_SMD:C_0402_1005Metric
- C3: value EEU-FM1V102 -> 100n; footprint Capacitor_THT:CP_Radial_D12.5mm_P5.00mm -> Capacitor_SMD:C_0603_1608Metric
- J3: value Conn_02x05_Counter_Clockwise -> RJ45_LED_Shielded; footprint Connector_IDC:IDC-Header_2x05_P2.54mm_Horizontal -> Library:MTJ-88ARX1-FSM-PG-LH
- J4: renamed from J2; value TBP04R12-500-04BE -> Conn_01x02; footprint Connector_Phoenix_MSTB:PhoenixContact_MSTBA_2,5_4-G_1x04_P5.00mm_Horizontal -> Connector_Phoenix_MSTB:PhoenixContact_MSTBA_2,5_2-G-5,08_1x02_P5.08mm_Horizontal
- J6: renamed from J5; value Conn_01x02 -> Conn_01x06_Socket; footprint Connector_JST:JST_XH_B2B-XH-A_1x02_P2.50mm_Vertical -> Connector_PinHeader_2.54mm:PinHeader_1x06_P2.54mm_Vertical
- JP1: value Jumper_3_Open -> Jumper_2_Small_Open; footprint Connector_PinHeader_2.54mm:PinHeader_1x03_P2.54mm_Vertical -> PCM_4ms_SolderJumper:JUMPER_SMD_1x2_tiny
- R11: renamed from R33; footprint Resistor_SMD:R_0603_1608Metric -> Resistor_SMD:R_0402_1005Metric
- R13: renamed from R7; footprint Resistor_SMD:R_0603_1608Metric -> Resistor_SMD:R_0402_1005Metric
- R16: renamed from R2; footprint Resistor_SMD:R_0603_1608Metric -> Resistor_SMD:R_0402_1005Metric
- R17: renamed from R3; footprint Resistor_SMD:R_0603_1608Metric -> Resistor_SMD:R_0402_1005Metric
- R18: renamed from R1; footprint Resistor_SMD:R_0603_1608Metric -> Resistor_SMD:R_0402_1005Metric
- R19: renamed from R4; footprint Resistor_SMD:R_0603_1608Metric -> Resistor_SMD:R_0402_1005Metric
- R20: renamed from R21; footprint Resistor_SMD:R_0603_1608Metric -> Resistor_SMD:R_0402_1005Metric
- R21: renamed from R13; footprint Resistor_SMD:R_0603_1608Metric -> Resistor_SMD:R_0402_1005Metric
- R22: renamed from R10; footprint Resistor_SMD:R_0603_1608Metric -> Resistor_SMD:R_0402_1005Metric
- R23: renamed from R5; footprint Resistor_SMD:R_0603_1608Metric -> Resistor_SMD:R_0402_1005Metric
- R24: renamed from R6; footprint Resistor_SMD:R_0603_1608Metric -> Resistor_SMD:R_0402_1005Metric
- R25: renamed from R12; footprint Resistor_SMD:R_0603_1608Metric -> Resistor_SMD:R_0402_1005Metric
- R26: renamed from R14; footprint Resistor_SMD:R_0603_1608Metric -> Resistor_SMD:R_0402_1005Metric
- R4: renamed from R35; footprint Resistor_SMD:R_0603_1608Metric -> Resistor_SMD:R_0402_1005Metric
- R5: renamed from R36; footprint Resistor_SMD:R_0603_1608Metric -> Resistor_SMD:R_0402_1005Metric
- U1: value COMPARATOR -> TPS22810DBV; footprint Library:COMPARATOR -> Package_TO_SOT_SMD:SOT-23-6
- moved J6 86.5 mm to (162.3, 115.0), turned to 180 degrees
- moved U1 48.5 mm to (110.7, 75.9), turned to -90 degrees
- moved JP1 41.0 mm to (85.2, 75.1), turned to 180 degrees
- moved J4 29.9 mm to (153.9, 86.7)
- moved J1 21.7 mm to (90.1, 75.2), turned to -90 degrees
- moved C18 16.6 mm to (103.2, 98.5)
- moved R12 13.8 mm to (155.8, 74.8)
- moved C4 13.3 mm to (121.4, 83.9), turned to -90 degrees
- moved D2 10.7 mm to (113.1, 81.9), turned to 90 degrees
- moved R4 10.5 mm to (88.5, 101.0), turned to 180 degrees
- moved C5 8.70 mm to (119.0, 83.9), turned to -90 degrees
- moved R11 8.63 mm to (113.1, 79.4), turned to 90 degrees
- moved C3 8.23 mm to (110.7, 78.9), turned to 0 degrees
- moved C9 8.10 mm to (152.5, 92.2), turned to 180 degrees
- moved R5 8.10 mm to (88.5, 100.0), turned to 180 degrees
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- renumbered C7 to C6, C2 to C8, C13 to C9, D2 to D1, D17 to D2, D1 to D3, D3 to D4, D4 to D5, D5 to D6, FB2 to FB1, FB1 to FB2, H4 to H3, J6 to J1, J4 to J5, R37 to R1, R19 to R12, R15 to R27, R11 to R28, R16 to R6, R20 to R9, U5 to U6
Connections:
- C17 pad 2: /VIN -> /VIN_SW
- C18 pad 2: /VIN -> /VIN_SW
- C3 pad 1: /VIN -> GND
- C3 pad 2: GND -> /VIN_SW
- C4 pad 1: /VIN -> /VIN_SW
- C5 pad 1: /VIN -> /VIN_SW
- C9 pad 1: Net-(J1-Pin_1) -> Net-(J4-Pin_1)
- C9 pad 2: Net-(C13-Pad2) -> /Comparator/IN
- J1 pad 1: Net-(D25-K) -> /VIN
- J3 pad 1: /PSU_EN1 -> GND
- J3 pad 10: /SCL -> unconnected-(J3-Pad10)
- J3 pad 2: /PWR_EN -> /VIN_RJ
- J3 pad 3: +3.3V -> GND
- J3 pad 4: +5V -> /PWR_EN
- J3 pad 5: GND -> /PSU_EN
- J3 pad 6: /GEIGER_OUTPUT -> /VIN_RJ
- J3 pad 7: /R1 -> /A
- J3 pad 8: /R2 -> /B
- J3 pad 9: /SDA -> unconnected-(J3-Pad9)
- J4 pad 1: GND -> Net-(J4-Pin_1)
- J6 pad 1: Net-(D25-K) -> unconnected-(J6-Pin_1-Pad1)
- J6 pad 2: GND -> /Pulse CNT/UPDI
- JP1 pad 1: /PSU_EN1 -> /VIN
- JP1 pad 2: /PSU_EN -> /VIN_RJ
- R11 pad 2: /VIN -> Net-(JP5-A)
- R12 pad 2: Net-(J1-Pin_1) -> Net-(J4-Pin_1)
- R16 pad 2: GND -> Net-(JP7-B)
- R17 pad 2: GND -> Net-(JP8-B)
- R27 pad 1: /VIN -> /VIN_SW
- R4 pad 2: +3.3V -> +5V
- R5 pad 2: +3.3V -> +5V
- U1 pad 1: +5V -> /VIN
- U1 pad 2: unconnected-(U1-~{OUT}-Pad2) -> GND
- U1 pad 3: /GEIGER_OUTPUT -> /PWR_EN
- U1 pad 4: GND -> Net-(U1-CT)
- U1 pad 5: Net-(C13-Pad2) -> /VIN_SW
- U1 pad 6: Net-(C13-Pad2) -> /VIN_SW
- U2 pad 3: /VIN -> /VIN_SW
- U2 pad 4: /VIN -> /VIN_SW
- U2 pad 5: /VIN -> /VIN_SW
- U2 pad 6: /VIN -> /VIN_SW
- U6 pad 12: unconnected-(U5-PB0-Pad12) -> /ADDR0
- U6 pad 14: unconnected-(U5-PB2-Pad14) -> /ADDR1
- U6 pad 2: /R1 -> /RE/DE
- U6 pad 30: /SW2 -> /R
- U6 pad 31: /SW3 -> /D
- U6 pad 7: /SW0 -> /ADDR2
- U6 pad 8: /SW1 -> /ADDR3
- U6 pad 9: /R2 -> /LINK
- U8 pad 1: /VIN -> /VIN_SW
- U8 pad 8: /VIN -> /VIN_SW
Routing:
- net +5V: track 216.8 -> 0.00 mm, vias 11 -> 0
- net /GEIGER_OUTPUT: track 88.9 -> 0.00 mm
- net /switcher/AD0: track 57.9 -> 0.00 mm, vias 2 -> 0
- net Net-(J1-Pin_1): track 44.2 -> 0.00 mm
- net GND: track 37.1 -> 0.00 mm, vias 42 -> 0
- net /PWR_EN: track 36.5 -> 0.00 mm, vias 3 -> 0
- net /switcher/RST: track 30.5 -> 0.00 mm, vias 2 -> 0
- net /switcher/AIN1: track 27.0 -> 0.00 mm
- net /VIN: track 24.4 -> 0.00 mm, vias 2 -> 0
- net /R2: track 19.7 -> 0.00 mm, vias 2 -> 0
- net +3.3V: track 18.6 -> 0.00 mm, vias 1 -> 0
- net /SCL: track 14.1 -> 0.00 mm
- net /R1: track 12.9 -> 0.00 mm, vias 2 -> 0
- net /switcher/SCK: track 12.8 -> 0.00 mm
- net /switcher/MISO: track 12.2 -> 0.00 mm, vias 2 -> 0
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- removed copper zone on F.Cu, net /VIN
- removed copper zone on F.Cu, net /switcher/T-
- removed copper zone on B.Cu, net GND
- removed copper zone on F.Cu, net GND
- removed copper zone on F.Cu, net Net-(D1-A)
- removed copper zone on B.Cu, net Net-(D1-K)
- removed copper zone on F.Cu, net Net-(D1-K)
- removed copper zone on F.Cu, net Net-(D25-K)
- removed copper zone on F.Cu, net Net-(D6-A2)
Other:
- board size 100 x 48 mm -> 94.1 x 48 mm
- board text removed: "+VIN"
- board text removed: "GND"
- board text removed: "↑A"
- board text removed: "↓C"
