File: pcb/RaSensLite/RaSensLite.kicad_sch (KiCad schematic)
At the start: 39 parts, among them J1 TBP04R12-500-04BE, J2 TBP04R12-500-04BE, J3 Conn_02x05_Counter_Clockwise, J5 Conn_01x02, J6 Conn_01x02, K5 DIP12-1A72-11L, Q15 2N2222A, U1 COMPARATOR, U2 DA2032-AL, U3 LM311

Commit message: d
Parts:
- removed C10: 100n, Capacitor_SMD:C_0805_2012Metric, symbol Device:C
- removed C14: 250p, Capacitor_SMD:C_1206_3216Metric, symbol Device:C
- removed D23, D24: BAS21, Diode_SMD:D_SOD-123F, symbol Device:D
- removed R25: 200k, Resistor_SMD:R_0805_2012Metric, symbol Device:R
- removed R26: 2Meg, Resistor_SMD:R_0805_2012Metric, symbol Device:R
- removed R27: 3Meg, Resistor_SMD:R_0805_2012Metric, symbol Device:R
- removed R34: 1k, Resistor_SMD:R_0603_1608Metric, symbol Device:R
- removed U3: LM311, Package_DIP:DIP-8_W7.62mm_Socket, symbol Comparator:LM311
Connections:
- no-connect marks 3 -> 1
Other:
- title: Geiger Counter Module -> RaSensLite
- moved on the sheet: H1, H2
