File: pcb/RaSensLite/RaSensLite.kicad_sch (KiCad schematic)
At the start: 37 parts, among them J1 TBP04R12-500-04BE, J2 TBP04R12-500-04BE, J3 Conn_02x05_Counter_Clockwise, J6 TBP04R12-500-02BE, K5 DIP12-1A72-11L, Q15 2N2222A, U2 DA2032-AL, U3 LM311

Commit message: V5
Parts:
- removed C8: EFDKA1CK105D032LH, Capacitor_THT:C_Rect_L31.5mm_W11.0mm_P27.50mm_MKS4, symbol Device:C
- removed J6: TBP04R12-500-02BE, Connector_Phoenix_MSTB:PhoenixContact_MSTBA_2,5_2-G-5,08_1x02_P5.08mm_Horizontal, symbol Connector:Screw_Terminal_01x02
- added C2: ECW-FD2J105PQ, Capacitor_THT:C_Rect_L18.0mm_W7.0mm_P15.00mm_FKS3_FKP3, symbol Device:C
- added J5, J6: Conn_01x02, Connector_JST:JST_XH_B2B-XH-A_1x02_P2.50mm_Vertical, symbol Connector_Generic:Conn_01x02
- added U1: COMPARATOR, Library:COMPARATOR, symbol library:Comparator
Connections:
- net +5V: now also U1.1 (+5V)
- net GEIGER_OUTPUT: now also U1.3 (OUT)
- net GND: now also C2.2, J5.2 (Pin_2), J6.2 (Pin_2), U1.4 (GND)
- net SCL: now also J3.10 (Pin_10); no longer J3.9 (Pin_9)
- net SDA: now also J3.9 (Pin_9); no longer J3.10 (Pin_10)
- net at C14.2, D24.1 (K), R25.2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: no longer C13.2
- net at D25.1 (K), K5.1, K5.14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: now also J5.1 (Pin_1), J6.1 (Pin_1)
- net at C7.2, D2.1 (K), R19.1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: now also C2.1
- new net: C13.2, U1.5 (IN), U1.6 (IN), U1.7 (IN), U1.8 (IN)
- no-connect marks 2 -> 3
Other:
- moved on the sheet: C10, C14, D23, D24, R25, R26, R27, R34, U3

Commit message: PCB 485
Parts:
- removed D23, D24: BAS21, Diode_SMD:D_SOD-123F, symbol Device:D
- removed D25: UF4007, Diode_THT:D_DO-41_SOD81_P10.16mm_Horizontal, symbol Diode:BA157
- removed J3: Conn_02x05_Counter_Clockwise, Connector_IDC:IDC-Header_2x05_P2.54mm_Horizontal, symbol Connector_Generic:Conn_02x05_Counter_Clockwise
- removed J5: Conn_01x02, Connector_JST:JST_XH_B2B-XH-A_1x02_P2.50mm_Vertical, symbol Connector_Generic:Conn_01x02
- removed JP1: Jumper_3_Open, Connector_PinHeader_2.54mm:PinHeader_1x03_P2.54mm_Vertical, symbol Jumper:Jumper_3_Open
- removed K5: DIP12-1A72-11L, Relay_THT:Relay_StandexMeder_DIP_LowProfile, symbol Relay:DIPxx-1Axx-11x
- removed Q15: 2N2222A, Package_TO_SOT_THT:TO-92L_Inline, symbol Transistor_BJT:BC107
- removed R25: 200k, Resistor_SMD:R_0805_2012Metric, symbol Device:R
- removed R26: 2Meg, Resistor_SMD:R_0805_2012Metric, symbol Device:R
- removed R27: 3Meg, Resistor_SMD:R_0805_2012Metric, symbol Device:R
- removed R34: 1k, Resistor_SMD:R_0603_1608Metric, symbol Device:R
- removed R46: 1k, Resistor_SMD:R_0805_2012Metric, symbol Device:R
- removed U3: LM311, Package_DIP:DIP-8_W7.62mm_Socket, symbol Comparator:LM311
- added C8: 100n, Capacitor_SMD:C_0603_1608Metric, symbol Device:C
- added J3, J8: RJ45_LED_Shielded, symbol Connector:RJ45_LED_Shielded
- added JP1, JP2, JP3, JP4, JP5: Jumper_2_Small_Open, PCM_4ms_SolderJumper:JUMPER_SMD_1x2_tiny, symbol Jumper:Jumper_2_Small_Open
- added R22, R23: 1k, Resistor_SMD:R_0603_1608Metric, symbol Device:R
- added R24: 120, Resistor_SMD:R_0603_1608Metric, symbol Device:R
- added R8, R9: 0, Resistor_SMD:R_0603_1608Metric, symbol Device:R
- added SW1: SW_DIP_x04, symbol Switch:SW_DIP_x04
- added U10: SN65HVD1781, Package_SO:SOIC-8_3.9x4.9mm_P1.27mm, symbol Interface_UART:SN65HVD1781
- added U3: TPS22810DBV, Package_TO_SOT_SMD:SOT-23-6, symbol Power_Management:TPS22810DBV
- C10: footprint Capacitor_SMD:C_0805_2012Metric -> Capacitor_SMD:C_0603_1608Metric
- C14: value 250p -> 2n2; footprint Capacitor_SMD:C_1206_3216Metric -> Capacitor_SMD:C_0603_1608Metric; now fitted; now in the parts list
Connections:
- net +3.3V is gone; now on net +5V: R35.2, R36.2
- net +5V: now also C8.2, U10.8 (VCC); no longer C10.2, C14.1
- net GND: now also C14.1, C8.1, J3.1, J3.3, J8.1, J8.3, JP3.2 (B), JP4.2 (B), SW1.5, SW1.6, SW1.7, SW1.8, U10.5 (GND), U3.2 (GND)
- net PSU_EN: now also J3.5, J8.5
- net PWR_EN: now also J3.4, J8.4, U3.3 (EN/UVLO)
- net VIN: now also J6.1 (Pin_1), JP1.1 (A), JP2.2 (B), U3.1 (VIN); no longer C4.1, C5.1, R33.2, U2.3, U2.4, U2.5, U2.6
- net at C14.2: now also U3.4 (CT)
- new net: JP2.1 (A), R33.2
- new net: JP3.1 (A), R22.1
- new net: J8.11, R22.2
- new net: J8.9, R23.2
- new net: R8.2, U10.1 (R)
- new net: JP5.2 (B), R24.2
- new net: JP4.1 (A), R23.1
- new net: R9.1, U10.4 (D)
- new net A: J3.7, J8.7, R24.1, U10.6 (A)
- new net ADDR0: SW1.1
- new net ADDR1: SW1.2
- new net ADDR2: SW1.3
- new net ADDR3: SW1.4
- new net B: J3.8, J8.8, JP5.1 (A), U10.7 (B)
- new net D: R9.2
- new net LINK: J8.12
- new net R: R8.1
- new net RE/DE: J8.10, U10.2 (~{RE}), U10.3 (DE)
- new net VIN_RJ: J3.2, J3.6, J8.2, J8.6, JP1.2 (B)
- new net VIN_SW: C10.2, C4.1, C5.1, U2.3, U2.4, U2.5, U2.6, U3.5 (QOD), U3.6 (VOUT)
- no-connect marks 3 -> 5
Other:
- added sheet Pulse CNT (pulseCnt.kicad_sch)
- sheet switcher ports: added ADDR0, ADDR1, ADDR2, ADDR3, LINK, RE/DE, RXD, TXD; removed RANGE0, RANGE1, R_SW0, R_SW1, R_SW2, R_SW3
- note added: "G"
- note added: "Y"
- moved on the sheet: C3, C4, C5, D17, H1, H2, H4, R33, R35, R36, U1

Commit message: v
Parts:
- removed C3: EEU-FM1V102, Capacitor_THT:CP_Radial_D12.5mm_P5.00mm, symbol Device:C_Polarized
- removed J1, J2: TBP04R12-500-04BE, Connector_Phoenix_MSTB:PhoenixContact_MSTBA_2,5_4-G_1x04_P5.00mm_Horizontal, symbol Connector:Screw_Terminal_01x04
- removed U1: COMPARATOR, Library:COMPARATOR, symbol library:Comparator
- added C10: EEE-FN1C102UP, Capacitor_SMD:CP_Elec_10x10.5, symbol Device:C_Polarized
- added J4: Conn_01x02, Connector_Phoenix_MSTB:PhoenixContact_MSTBA_2,5_2-G-5,08_1x02_P5.08mm_Horizontal, symbol Connector_Generic:Conn_01x02
- added JP6: Jumper_2_Open, TestPoint:TestPoint_2Pads_Pitch2.54mm_Drill0.8mm, symbol Jumper:Jumper_2_Open
- C7: renamed from C8; footprint Capacitor_SMD:C_0603_1608Metric -> Capacitor_SMD:C_0402_1005Metric
- J2: renamed from J8; footprint (none) -> Library:MTJ-88ARX1-FSM-PG-LH
- J3: footprint (none) -> Library:MTJ-88ARX1-FSM-PG-LH
- R11: renamed from R33; footprint Resistor_SMD:R_0603_1608Metric -> Resistor_SMD:R_0402_1005Metric
- R2: renamed from R23; footprint Resistor_SMD:R_0603_1608Metric -> Resistor_SMD:R_0402_1005Metric
- R3: renamed from R22; footprint Resistor_SMD:R_0603_1608Metric -> Resistor_SMD:R_0402_1005Metric
- R4: renamed from R35; footprint Resistor_SMD:R_0603_1608Metric -> Resistor_SMD:R_0402_1005Metric
- R5: renamed from R36; footprint Resistor_SMD:R_0603_1608Metric -> Resistor_SMD:R_0402_1005Metric
- SW1: footprint (none) -> Button_Switch_SMD:SW_DIP_SPSTx04_Slide_6.7x11.72mm_W6.73mm_P2.54mm_LowProfile_JPin
- renumbered C14 to C2, C10 to C3, C7 to C6, C2 to C8, C13 to C9, D2 to D1, D17 to D2, H4 to H3, J6 to J1, JP4 to JP2, JP5 to JP4, JP2 to JP5, R37 to R1, R24 to R10, R19 to R12, R16 to R6, R8 to R7, R9 to R8, R20 to R9, U3 to U1, U10 to U3
Connections:
- net ADDR0: now also SW1.2; no longer SW1.1
- net ADDR1: now also SW1.1; no longer SW1.2
- net ADDR2: now also SW1.4; no longer SW1.3
- net ADDR3: now also SW1.3; no longer SW1.4
- net GEIGER_OUTPUT: now also JP6.1 (A)
- net GND: now also C10.2, J4.2 (Pin_2)
- net VIN: now also C10.1; no longer JP5.2 (B)
- net VIN_SW: now also JP5.2 (B)
- net at C9.1, R12.2: now also J4.1 (Pin_1)
- net Comparator/IN: now reaches C9.2
- new net Comparator/OUT: JP6.2 (B)
- no-connect marks 5 -> 4
Other:
- added sheet Comparator (comp.kicad_sch)
- moved on the sheet: C7, J2, J3, JP1, JP2, JP3, JP4, R10, R2, R3, R7, R8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
