File: pcb/RaSensLite/switcher.kicad_sch (KiCad schematic)
At the start: 41 parts, among them J4 TC2030, Q1 IPP075N15N3, U4 LM4040DBZ-2.5, U5 ATmega328P-A, U6 LM317_SOT-223, U7 LM321, U8 TC4420, U9 LM321

Commit message: d
Other:
- title: Geiger Counter Module -> RaSensLite
Changed lines of the file:
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@@
 	(paper "A4")
 	(title_block
-		(title "Geiger Counter Module")
-		(date "2025-09-16")
-		(rev "A")
+		(title "RaSensLite")
+		(date "2026-05-17")
+		(rev "v5")
 	)
 	(text "FB AMP\n"
