File: pcb/RaSensLite/switcher.kicad_sch (KiCad schematic)
At the start: 41 parts, among them J4 TC2030, Q1 IPP075N15N3, U4 LM4040DBZ-2.5, U5 ATmega328P-A, U6 LM317_SOT-223, U7 LM321, U8 TC4420, U9 LM321

Commit message: PCB 485
Parts:
- added JP6, JP7: Jumper_2_Small_Open, PCM_4ms_SolderJumper:JUMPER_SMD_1x2_tiny, symbol Jumper:Jumper_2_Small_Open
Connections:
- net GND: now also JP6.1 (A), JP7.1 (A); no longer R2.2, R3.2
- net ADDR0: now reaches U5.12 (PB0)
- net ADDR1: now reaches U5.14 (PB2)
- net RANGE0 renamed RE/DE
- net RANGE1 renamed LINK
- net R_SW0 renamed ADDR2
- net R_SW1 renamed ADDR3
- net R_SW2 renamed RXD
- net R_SW3 renamed TXD
- new net: JP6.2 (B), R2.2
- new net: JP7.2 (B), R3.2
Changed lines of the file:
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@@
 	)
 	(junction
-		(at 101.6 179.07)
-		(diameter 0)
-		(color 0 0 0 0)
-	)
-	(junction
 		(at 55.88 127)
 		(diameter 0)
@@
 	)
 	(junction
+		(at 106.68 179.07)
+		(diameter 0)
+		(color 0 0 0 0)
+	)
+	(junction
 		(at 185.42 127)
 		(diameter 0)
@@
 	(wire
 		(pts
-			(xy 99.06 179.07) (xy 101.6 179.07)
+			(xy 99.06 179.07) (xy 100.33 179.07)
 		)
 		(stroke
@@
 	(wire
 		(pts
-			(xy 99.06 91.44) (xy 107.95 91.44)
-		)
-		(stroke
-			(width 0)
-			(type default)
-		)
-	)
-	(wire
-		(pts
 			(xy 116.84 111.76) (xy 116.84 110.49)
 		)
@@
 	(wire
 		(pts
-			(xy 101.6 167.64) (xy 99.06 167.64)
+			(xy 100.33 167.64) (xy 99.06 167.64)
 		)
 		(stroke
@@
 	(wire
 		(pts
+			(xy 106.68 179.07) (xy 106.68 167.64)
+		)
+		(stroke
+			(width 0)
+			(type default)
+		)
+	)
+	(wire
+		(pts
 			(xy 242.57 146.05) (xy 242.57 147.32)
 		)
@@
 	(wire
 		(pts
+			(xy 106.68 167.64) (xy 105.41 167.64)
+		)
+		(stroke
+			(width 0)
+			(type default)
+		)
+	)
+	(wire
+		(pts
 			(xy 21.59 127) (xy 21.59 128.27)
 		)
@@
 	(wire
 		(pts
-			(xy 101.6 179.07) (xy 101.6 167.64)
+			(xy 99.06 73.66) (xy 107.95 73.66)
 		)
 		(stroke
@@
 	(wire
 		(pts
+			(xy 99.06 88.9) (xy 107.95 88.9)
+		)
+		(stroke
+			(width 0)
+			(type default)
+		)
+	)
+	(wire
+		(pts
 			(xy 88.9 35.56) (xy 88.9 36.83)
 		)
@@
 	(wire
 		(pts
+			(xy 99.06 91.44) (xy 107.95 91.44)
+		)
+		(stroke
+			(width 0)
+			(type default)
+		)
+	)
+	(wire
+		(pts
 			(xy 99.06 132.08) (xy 107.95 132.08)
 		)
@@
 	(wire
 		(pts
-			(xy 99.06 88.9) (xy 107.95 88.9)
+			(xy 106.68 181.61) (xy 106.68 179.07)
 		)
 		(stroke
@@
 	(wire
 		(pts
+			(xy 105.41 179.07) (xy 106.68 179.07)
+		)
+		(stroke
+			(width 0)
+			(type default)
+		)
+	)
+	(wire
+		(pts
 			(xy 78.74 58.42) (xy 83.82 58.42)
 		)
@@
 	(wire
 		(pts
-			(xy 101.6 181.61) (xy 101.6 179.07)
-		)
-		(stroke
-			(width 0)
-			(type default)
-		)
-	)
-	(wire
-		(pts
 			(xy 46.99 146.05) (xy 46.99 148.59)
 		)
@@
 	(wire
 		(pts
+			(xy 99.06 78.74) (xy 107.95 78.74)
+		)
+		(stroke
+			(width 0)
+			(type default)
+		)
+	)
+	(wire
+		(pts
 			(xy 229.87 86.36) (xy 246.38 86.36)
 		)
@@
 		)
 	)
-	(hierarchical_label "RANGE1"
+	(hierarchical_label "ADDR0"
+		(shape output)
+		(at 107.95 73.66 0)
+		(effects
+			(font
+				(size 1.27 1.27)
+			)
+			(justify left)
+		)
+	)
+	(hierarchical_label "LINK"
 		(shape input)
 		(at 107.95 129.54 0)
@@
 		)
 	)
-	(hierarchical_label "R_SW3"
+	(hierarchical_label "TXD"
 		(shape output)
 		(at 107.95 119.38 0)
@@
 		)
 	)
-	(hierarchical_label "RANGE0"
+	(hierarchical_label "ADDR1"
+		(shape output)
+		(at 107.95 78.74 0)
+		(effects
+			(font
+				(size 1.27 1.27)
+			)
+			(justify left)
+		)
+	)
+	(hierarchical_label "RE{slash}DE"
 		(shape input)
 		(at 107.95 127 0)
@@
 		)
 	)
+	(hierarchical_label "ADDR2"
+		(shape output)
+		(at 107.95 88.9 0)
+		(effects
+			(font
+				(size 1.27 1.27)
+			)
+			(justify left)
+		)
+	)
 	(hierarchical_label "VIN"
 		(shape passive)
@@
 		)
 	)
-	(hierarchical_label "R_SW2"
-		(shape output)
+	(hierarchical_label "RXD"
+		(shape input)
 		(at 107.95 116.84 0)
 		(effects
@@
 		)
 	)
-	(hierarchical_label "R_SW1"
+	(hierarchical_label "ADDR3"
 		(shape output)
 		(at 107.95 91.44 0)
@@
 		)
 	)
-	(hierarchical_label "R_SW0"
-		(shape output)
-		(at 107.95 88.9 0)
-		(effects
-			(font
-				(size 1.27 1.27)
-			)
-			(justify left)
-		)
-	)
 	(symbol
 		(lib_id "Connector:TC2030")
@@
 	)
 	(symbol
+		(lib_id "Jumper:Jumper_2_Small_Open")
+		(at 102.87 167.64 0)
+		(mirror y)
+		(unit 1)
+		(exclude_from_sim no)
+		(in_bom yes)
+		(on_board yes)
+		(dnp no)
+		(fields_autoplaced yes)
+		(property "Reference" "JP6"
+			(at 102.87 163.83 0)
+			(effects
+				(font
+					(size 1.27 1.27)
+				)
+			)
+		)
+		(property "Value" "Jumper_2_Small_Open"
+			(at 104.1399 168.91 90)
+			(effects
+				(font
+					(size 1.27 1.27)
+				)
+				(justify right)
+				(hide yes)
+			)
+		)
+		(property "Footprint" "PCM_4ms_SolderJumper:JUMPER_SMD_1x2_tiny"
+			(at 102.87 167.64 0)
+			(effects
+				(font
+					(size 1.27 1.27)
+				)
+				(hide yes)
+			)
+		)
+		(property "Datasheet" "~"
+			(at 102.87 167.64 0)
+			(effects
+				(font
+					(size 1.27 1.27)
+				)
+				(hide yes)
+			)
+		)
+		(property "Description" "Jumper, 2-pole, small symbol, open"
+			(at 102.87 167.64 0)
+			(effects
+				(font
+					(size 1.27 1.27)
+				)
+				(hide yes)
+			)
+		)
+		(pin "2"
+		)
+		(pin "1"
+		)
+		(instances
+			(project "RaSensLite"
+				(path "/5a813425-ce65-4d1a-8158-1ddcc9c68fab/45aa0ff5-e54f-42d4-9b38-b99b85e204b5"
+					(reference "JP6")
+					(unit 1)
+				)
+			)
+		)
+	)
+	(symbol
 		(lib_id "Device:C")
 		(at 242.57 151.13 0)
@@
 	)
 	(symbol
+		(lib_id "Jumper:Jumper_2_Small_Open")
+		(at 102.87 179.07 0)
+		(mirror y)
+		(unit 1)
+		(exclude_from_sim no)
+		(in_bom yes)
+		(on_board yes)
+		(dnp no)
+		(fields_autoplaced yes)
+		(property "Reference" "JP7"
+			(at 102.87 175.26 0)
+			(effects
+				(font
+					(size 1.27 1.27)
+				)
+			)
+		)
+		(property "Value" "Jumper_2_Small_Open"
+			(at 104.1399 180.34 90)
+			(effects
+				(font
+					(size 1.27 1.27)
+				)
+				(justify right)
+				(hide yes)
+			)
+		)
+		(property "Footprint" "PCM_4ms_SolderJumper:JUMPER_SMD_1x2_tiny"
+			(at 102.87 179.07 0)
+			(effects
+				(font
+					(size 1.27 1.27)
+				)
+				(hide yes)
+			)
+		)
+		(property "Datasheet" "~"
+			(at 102.87 179.07 0)
+			(effects
+				(font
+					(size 1.27 1.27)
+				)
+				(hide yes)
+			)
+		)
+		(property "Description" "Jumper, 2-pole, small symbol, open"
+			(at 102.87 179.07 0)
+			(effects
+				(font
+					(size 1.27 1.27)
+				)
+				(hide yes)
+			)
+		)
+		(pin "2"
+		)
+		(pin "1"
+		)
+		(instances
+			(project "RaSensLite"
+				(path "/5a813425-ce65-4d1a-8158-1ddcc9c68fab/45aa0ff5-e54f-42d4-9b38-b99b85e204b5"
+					(reference "JP7")
+					(unit 1)
+				)
+			)
+		)
+	)
+	(symbol
 		(lib_id "Device:C")
 		(at 256.54 151.13 0)
@@
 	(symbol
 		(lib_id "power:GND")
-		(at 101.6 181.61 0)
+		(at 106.68 181.61 0)
 		(mirror y)
 		(unit 1)
@@
 		(on_board yes)
 		(dnp no)
-		(fields_autoplaced yes)
 		(property "Reference" "#PWR014"
-			(at 101.6 187.96 0)
+			(at 106.68 187.96 0)
 			(effects
 				(font
@@
 		)
 		(property "Value" "GND"
-			(at 101.6 186.69 0)
+			(at 106.68 185.166 0)
 			(effects
 				(font
@@
 		)
 		(property "Footprint" ""
-			(at 101.6 181.61 0)
+			(at 106.68 181.61 0)
 			(effects
 				(font
@@
 		)
 		(property "Datasheet" ""
-			(at 101.6 181.61 0)
+			(at 106.68 181.61 0)
 			(effects
 				(font
@@
 		)
 		(property "Description" "Power symbol creates a global label with name \"GND\" , ground"
-			(at 101.6 181.61 0)
+			(at 106.68 181.61 0)
 			(effects
 				(font

Commit message: v
Parts:
- removed C11: 1u, Capacitor_SMD:C_0603_1608Metric, symbol Device:C
- removed C12: 10u, Capacitor_SMD:C_1206_3216Metric, symbol Device:C
- removed R17: 240, Resistor_SMD:R_0603_1608Metric, symbol Device:R
- removed R18: 720, Resistor_SMD:R_0603_1608Metric, symbol Device:R
- removed U6: LM317_SOT-223, Package_TO_SOT_SMD:SOT-223-3_TabPin2, symbol Regulator_Linear:LM317_SOT-223
- added C24: 1u, Capacitor_SMD:C_0402_1005Metric, symbol Device:C
- added C25, C28: 22u, Capacitor_SMD:C_1206_3216Metric, symbol Device:C
- added C26: 10p, Capacitor_SMD:C_0603_1608Metric, symbol Device:C
- added C27: 100n, Capacitor_SMD:C_0402_1005Metric, symbol Device:C
- added L1: LSANB2016KKT4R7M, Inductor_SMD:L_0805_2012Metric, symbol Device:L_Small
- added R38: 10, Resistor_SMD:R_0402_1005Metric, symbol Device:R
- added R39: 47k, Resistor_SMD:R_0402_1005Metric, symbol Device:R
- added R40: 7k68, Resistor_SMD:R_0603_1608Metric, symbol Device:R
- added R41: 40k2, Resistor_SMD:R_0603_1608Metric, symbol Device:R
- added R42: 100k, Resistor_SMD:R_0402_1005Metric, symbol Device:R
- added U12: MP1476, Package_TO_SOT_SMD:SOT-563, symbol library:MP1476
- C12: renamed from C6; footprint Capacitor_SMD:C_0603_1608Metric -> Capacitor_SMD:C_0402_1005Metric
- C13: renamed from C9; footprint Capacitor_SMD:C_0603_1608Metric -> Capacitor_SMD:C_0402_1005Metric
- C14: renamed from C1; footprint Capacitor_SMD:C_0603_1608Metric -> Capacitor_SMD:C_0402_1005Metric
- R13: renamed from R7; footprint Resistor_SMD:R_0603_1608Metric -> Resistor_SMD:R_0402_1005Metric
- R16: renamed from R2; footprint Resistor_SMD:R_0603_1608Metric -> Resistor_SMD:R_0402_1005Metric
- R17: renamed from R3; footprint Resistor_SMD:R_0603_1608Metric -> Resistor_SMD:R_0402_1005Metric
- R18: renamed from R1; footprint Resistor_SMD:R_0603_1608Metric -> Resistor_SMD:R_0402_1005Metric
- R19: renamed from R4; footprint Resistor_SMD:R_0603_1608Metric -> Resistor_SMD:R_0402_1005Metric
- R20: renamed from R21; footprint Resistor_SMD:R_0603_1608Metric -> Resistor_SMD:R_0402_1005Metric
- R21: renamed from R13; footprint Resistor_SMD:R_0603_1608Metric -> Resistor_SMD:R_0402_1005Metric
- R22: renamed from R10; footprint Resistor_SMD:R_0603_1608Metric -> Resistor_SMD:R_0402_1005Metric
- R23: renamed from R5; footprint Resistor_SMD:R_0603_1608Metric -> Resistor_SMD:R_0402_1005Metric
- R24: renamed from R6; footprint Resistor_SMD:R_0603_1608Metric -> Resistor_SMD:R_0402_1005Metric
- R25: renamed from R12; footprint Resistor_SMD:R_0603_1608Metric -> Resistor_SMD:R_0402_1005Metric
- R26: renamed from R14; footprint Resistor_SMD:R_0603_1608Metric -> Resistor_SMD:R_0402_1005Metric
- renumbered D1 to D3, D3 to D4, D4 to D5, D5 to D6, FB2 to FB1, FB1 to FB2, J4 to J5, JP6 to JP7, JP7 to JP8, R15 to R27, R11 to R28, U5 to U6
Connections:
- net +5V: now also C26.1, C28.2, L1.2, R41.1
- net GND: now also C25.1, C27.2, C28.1, R40.1, U12.3 (GND)
- net VIN: now also C25.2, C27.1, R42.2, U12.1 (IN)
- new net: C24.2, L1.1, U12.2 (SW)
- new net: R38.1, U12.4 (BST)
- new net: R42.1, U12.5 (EN)
- new net: R39.1, U12.6 (FB)
- new net: C26.2, R39.2, R40.2, R41.2
- new net: C24.1, R38.2
Other:
- moved on the sheet: D3, D4, JP7, JP8, R16, R17
