File: pcb/RaSensLite/comp.kicad_sch (KiCad schematic)
At the start: 9 parts, among them J6 Conn_01x06_Socket, U10 ATtiny412-SS

Commit message: v
Parts:
- removed C21: 100n, Capacitor_SMD:C_0402_1005Metric, symbol Device:C
- removed C22: 100p, Capacitor_SMD:C_0603_1608Metric, symbol Device:C
- removed D7: D_Schottky, Diode_SMD:D_SOD-323, symbol Device:D_Schottky
- removed J6: Conn_01x06_Socket, Connector_PinHeader_2.54mm:PinHeader_1x06_P2.54mm_Vertical, symbol Connector:Conn_01x06_Socket
- removed R29: 1k, Resistor_SMD:R_0402_1005Metric, symbol Device:R
- removed R30: 470, Resistor_SMD:R_0402_1005Metric, symbol Device:R
- removed R31: 330k, Resistor_SMD:R_0402_1005Metric, symbol Device:R
- removed R32: 1Meg, Resistor_SMD:R_0402_1005Metric, symbol Device:R
- removed U10: ATtiny412-SS, Package_SO:SOIC-8_3.9x4.9mm_P1.27mm, symbol MCU_Microchip_ATtiny:ATtiny412-SS
- added C23: 0u1, Capacitor_SMD:C_0402_1005Metric, symbol Device:C
- added D8, D9: 1N5819WS, Diode_SMD:D_SOD-323, symbol Diode:1N5819WS
- added R33: 1M, Resistor_SMD:R_0402_1005Metric, symbol Device:R
- added R34, R37: 100k, Resistor_SMD:R_0402_1005Metric, symbol Device:R
- added R35: 10k, Resistor_SMD:R_0402_1005Metric, symbol Device:R
- added R36: 59k, Resistor_SMD:R_0603_1608Metric, symbol Device:R
- added RV1: 3314J-1-504E, Potentiometer_SMD:Potentiometer_Bourns_3314J_Vertical, symbol Device:R_Potentiometer_Trim
- added U11: LT1711xMS8, Package_SO:MSOP-8_3x3mm_P0.65mm, symbol Comparator:LT1711xMS8
Connections:
- net +5V: now also C23.1, D8.1 (K), RV1.2, U11.1 (V+)
- net GND: now also C23.2, D9.2 (A), R34.2, R37.1, U11.4 (V-), U11.5 (LATCH), U11.6 (GND)
- new net: D8.2 (A), D9.1 (K), R33.2, R36.1, R37.2, U11.2 (+)
- new net: R34.1, R35.1, U11.3 (-)
- new net: R35.2, RV1.1
- new net IN: R36.2
- new net OUT: R33.1, U11.7 (Q)
- no-connect marks 3 -> 0
Other:
- title: (none) -> Geiger Counter Module
