File: pcb/Switcher/Switcher.kicad_sch (KiCad schematic)
At the start: 2 parts, among them J2 Conn_01x10_Pin, J3 Conn_01x10_Pin

Commit message: d
Other:
- title: Flyback Controller -> RaSens Pro - Switcher
Changed lines of the file:
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@@
 	(paper "A4")
 	(title_block
-		(title "Flyback Controller")
-		(date "2025-09-16")
-		(rev "A")
+		(title "RaSens Pro - Switcher")
+		(date "2026-05-17")
+		(rev "v1")
 	)
 	(junction
