File: pcb/Switcher/core.kicad_sch (KiCad schematic)
At the start: 42 parts, among them J1 TC2030, Q1 IPP075N15N3, U1 ATmega328P-A, U2 LM321, U3 LM4040DBZ-2.5, U4 LM321, U5 TC4420, U6 LM317_SOT-223

Commit message: d
Other:
- title: Flyback Controller -> RaSens Pro - Switcher
Changed lines of the file:
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@@
 	(paper "A4")
 	(title_block
-		(title "Flyback Controller")
-		(date "2025-09-16")
-		(rev "A")
+		(title "RaSens Pro - Switcher")
+		(date "2026-05-17")
+		(rev "v1")
 	)
 	(text "OC AMP\n"
